Commit message: Model belt as a driven prismatic joint (belt_moving) and wire gzfortress plugin

File: ev3_manipulator/urdf/manipulator_gazebo.xacro (robot description, xacro)
@@ -161,4 +161,18 @@
     <self_collide>false</self_collide>
   </gazebo>
+  <!-- High friction on the moving belt slab so objects grip and ride it. -->
+  <gazebo reference="belt_moving">
+    <mu1>100.0</mu1>
+    <mu2>100.0</mu2>
+    <kp>1e6</kp>
+    <kd>10.0</kd>
+    <self_collide>false</self_collide>
+  </gazebo>
+  <!-- Keep conveyor_belt_link_1 out of fixed-joint lumping so belt_moving_joint's
+       parent link survives the URDF->SDF conversion. -->
+  <gazebo reference="conveyor_link_linkage_joint">
+    <preserveFixedJoint>true</preserveFixedJoint>
+    <disableFixedJointLumping>true</disableFixedJointLumping>
+  </gazebo>
   <gazebo reference="conveyor_linkage_link_1">
     <material>${body_color}</material>
@@ -179,12 +193,17 @@
     <self_collide>false</self_collide>
   </gazebo>
-  <!-- <gazebo>
-    <plugin filename="libROS2ConveyorBeltPlugin.so" name="ros2_conveyorbelt_plugin">
-      <ros>
-          <namespace></namespace>
-      </ros>
-      <max_velocity>0.5</max_velocity> <publish_rate>10</publish_rate>
+  <!-- Conveyor belt (IFRA gzfortress System plugin). Drives belt_moving_joint's
+       velocity + resets its position at the 1cm limit → objects ride the belt.
+       Control via the CONVEYORPOWER service (0-100%). Old Gazebo-Classic
+       libROS2ConveyorBeltPlugin.so retired (won't load on Fortress). -->
+  <gazebo>
+    <plugin filename="libros2gz_conveyorbelt_system.so" name="ros2_conveyorbelt_system">
+      <joint_name>belt_moving_joint</joint_name>
+      <max_velocity>0.15</max_velocity>
+      <publish_rate>1000</publish_rate>
+      <lower_limit>0.0</lower_limit>
+      <upper_limit>0.01</upper_limit>
     </plugin>
-  </gazebo> -->
+  </gazebo>
   <gazebo>
     <plugin filename="gz_ros2_control-system"

File: ev3_manipulator/urdf/manipulator_urdf.xacro (robot description, xacro)
@@ -638,4 +638,29 @@
     <child link="conveyor_belt_link_1"/>
   </joint>
+  <!-- ===== Conveyor moving surface (IFRA gzfortress style) =====
+       Invisible thin high-friction slab that rides a prismatic joint. The
+       ros2gz_conveyorbelt_system plugin commands this joint's velocity and
+       resets its position at the 1cm limit, so objects ride the belt by
+       friction. Sized to the belt footprint; top set just above the belt mesh
+       (link-frame belt top ~0.039) so objects contact this slab, not scenery. -->
+  <link name="belt_moving">
+    <inertial>
+      <origin xyz="0 0 0" rpy="0 0 0"/>
+      <mass value="50.0"/>
+      <inertia ixx="1e-4" iyy="1e-4" izz="1e-4" ixy="0" ixz="0" iyz="0"/>
+    </inertial>
+    <collision>
+      <origin xyz="0 0 0" rpy="0 0 0"/>
+      <geometry><box size="0.37 0.065 0.002"/></geometry>
+    </collision>
+  </link>
+  <joint name="belt_moving_joint" type="prismatic">
+    <origin xyz="0.099 0.035 0.040" rpy="0 0 0"/>
+    <parent link="conveyor_belt_link_1"/>
+    <child link="belt_moving"/>
+    <axis xyz="1 0 0"/>   <!-- belt travels along +X (long axis) -->
+    <limit lower="0.0" upper="0.01" effort="1e8" velocity="10.0"/>
+    <dynamics damping="1.0" friction="0.0"/>
+  </joint>
   <joint name="left_pulley_shaft_motor_housing_shaft" type="continuous">
     <origin xyz="-0.123678 0.053 -0.017678" rpy="0 0 0"/>
