Commit message: manipulator_urdf.xacro: use package:// mesh URIs so remote RViz/Foxglove can resolve them

File: ev3_manipulator/urdf/manipulator_urdf.xacro (robot description, xacro)
@@ -23,5 +23,5 @@
       <origin xyz="0 0 0" rpy="0 0 0"/>
       <geometry>
-        <mesh filename="file://$(find ev3_manipulator)/meshes/base_link.stl" scale="0.001 0.001 0.001"/>
+        <mesh filename="package://ev3_manipulator/meshes/base_link.stl" scale="0.001 0.001 0.001"/>
       </geometry>
       <material name="silver"/>
@@ -30,5 +30,5 @@
       <origin xyz="0 0 0" rpy="0 0 0"/>
       <geometry>
-        <mesh filename="file://$(find ev3_manipulator)/meshes/base_link.stl" scale="0.001 0.001 0.001"/>
+        <mesh filename="package://ev3_manipulator/meshes/base_link.stl" scale="0.001 0.001 0.001"/>
       </geometry>
     </collision>
@@ -44,5 +44,5 @@
       <origin xyz="0.020125 -0.103583 -0.094" rpy="0 0 0"/>
       <geometry>
-        <mesh filename="file://$(find ev3_manipulator)/meshes/arm_1_1.stl" scale="0.001 0.001 0.001"/>
+        <mesh filename="package://ev3_manipulator/meshes/arm_1_1.stl" scale="0.001 0.001 0.001"/>
       </geometry>
       <material name="silver"/>
@@ -51,5 +51,5 @@
       <origin xyz="0.020125 -0.103583 -0.094" rpy="0 0 0"/>
       <geometry>
-        <mesh filename="file://$(find ev3_manipulator)/meshes/arm_1_1.stl" scale="0.001 0.001 0.001"/>
+        <mesh filename="package://ev3_manipulator/meshes/arm_1_1.stl" scale="0.001 0.001 0.001"/>
       </geometry>
     </collision>
@@ -65,5 +65,5 @@
       <origin xyz="0.055125 -0.038117 -0.204384" rpy="0 0 0"/>
       <geometry>
-        <mesh filename="file://$(find ev3_manipulator)/meshes/left_arm_linkage_1.stl" scale="0.001 0.001 0.001"/>
+        <mesh filename="package://ev3_manipulator/meshes/left_arm_linkage_1.stl" scale="0.001 0.001 0.001"/>
       </geometry>
       <material name="silver"/>
@@ -72,5 +72,5 @@
       <origin xyz="0.055125 -0.038117 -0.204384" rpy="0 0 0"/>
       <geometry>
-        <mesh filename="file://$(find ev3_manipulator)/meshes/left_arm_linkage_1.stl" scale="0.001 0.001 0.001"/>
+        <mesh filename="package://ev3_manipulator/meshes/left_arm_linkage_1.stl" scale="0.001 0.001 0.001"/>
       </geometry>
     </collision>
@@ -86,5 +86,5 @@
       <origin xyz="0.055125 -0.0374 -0.266626" rpy="0 0 0"/>
       <geometry>
-        <mesh filename="file://$(find ev3_manipulator)/meshes/arm_2_1.stl" scale="0.001 0.001 0.001"/>
+        <mesh filename="package://ev3_manipulator/meshes/arm_2_1.stl" scale="0.001 0.001 0.001"/>
       </geometry>
       <material name="silver"/>
@@ -93,5 +93,5 @@
       <origin xyz="0.055125 -0.0374 -0.266626" rpy="0 0 0"/>
       <geometry>
-        <mesh filename="file://$(find ev3_manipulator)/meshes/arm_2_1.stl" scale="0.001 0.001 0.001"/>
+        <mesh filename="package://ev3_manipulator/meshes/arm_2_1.stl" scale="0.001 0.001 0.001"/>
       </geometry>
     </collision>
@@ -107,5 +107,5 @@
       <origin xyz="0.027725 -0.264363 -0.266669" rpy="0 0 0"/>
       <geometry>
-        <mesh filename="file://$(find ev3_manipulator)/meshes/arm_2_connector_1.stl" scale="0.001 0.001 0.001"/>
+        <mesh filename="package://ev3_manipulator/meshes/arm_2_connector_1.stl" scale="0.001 0.001 0.001"/>
       </geometry>
       <material name="silver"/>
@@ -114,5 +114,5 @@
       <origin xyz="0.027725 -0.264363 -0.266669" rpy="0 0 0"/>
       <geometry>
-        <mesh filename="file://$(find ev3_manipulator)/meshes/arm_2_connector_1.stl" scale="0.001 0.001 0.001"/>
+        <mesh filename="package://ev3_manipulator/meshes/arm_2_connector_1.stl" scale="0.001 0.001 0.001"/>
       </geometry>
     </collision>
@@ -129,5 +129,5 @@
       <origin xyz="0.020224 -0.267275 -0.221038" rpy="0 0 0"/>
       <geometry>
-        <mesh filename="file://$(find ev3_manipulator)/meshes/arm_3_1.stl" scale="0.001 0.001 0.001"/>
+        <mesh filename="package://ev3_manipulator/meshes/arm_3_1.stl" scale="0.001 0.001 0.001"/>
       </geometry>
       <material name="silver"/>
@@ -136,5 +136,5 @@
       <origin xyz="0.020224 -0.267275 -0.221038" rpy="0 0 0"/>
       <geometry>
-        <mesh filename="file://$(find ev3_manipulator)/meshes/arm_3_1.stl" scale="0.001 0.001 0.001"/>
+        <mesh filename="package://ev3_manipulator/meshes/arm_3_1.stl" scale="0.001 0.001 0.001"/>
       </geometry>
     </collision>
@@ -153,5 +153,5 @@
       <origin xyz="0.019938 -0.309958 -0.147299" rpy="0 0 0"/>
       <geometry>
-        <mesh filename="file://$(find ev3_manipulator)/meshes/left_gear_link_1.stl" scale="0.001 0.001 0.001"/>
+        <mesh filename="package://ev3_manipulator/meshes/left_gear_link_1.stl" scale="0.001 0.001 0.001"/>
       </geometry>
       <material name="silver"/>
@@ -160,5 +160,5 @@
       <origin xyz="0.019938 -0.309958 -0.147299" rpy="0 0 0"/>
       <geometry>
-        <mesh filename="file://$(find ev3_manipulator)/meshes/left_gear_link_1.stl" scale="0.001 0.001 0.001"/>
+        <mesh filename="package://ev3_manipulator/meshes/left_gear_link_1.stl" scale="0.001 0.001 0.001"/>
       </geometry>
     </collision>
@@ -174,5 +174,5 @@
       <origin xyz="0.019938 -0.276958 -0.147299" rpy="0 0 0"/>
       <geometry>
-        <mesh filename="file://$(find ev3_manipulator)/meshes/right_gear_link_1.stl" scale="0.001 0.001 0.001"/>
+        <mesh filename="package://ev3_manipulator/meshes/right_gear_link_1.stl" scale="0.001 0.001 0.001"/>
       </geometry>
       <material name="silver"/>
@@ -181,5 +181,5 @@
       <origin xyz="0.019938 -0.276958 -0.147299" rpy="0 0 0"/>
       <geometry>
-        <mesh filename="file://$(find ev3_manipulator)/meshes/right_gear_link_1.stl" scale="0.001 0.001 0.001"/>
+        <mesh filename="package://ev3_manipulator/meshes/right_gear_link_1.stl" scale="0.001 0.001 0.001"/>
       </geometry>
     </collision>
@@ -195,5 +195,5 @@
       <origin xyz="0.04992 -0.305958 -0.147299" rpy="0 0 0"/>
       <geometry>
-        <mesh filename="file://$(find ev3_manipulator)/meshes/left_finger_inner_link_1.stl" scale="0.001 0.001 0.001"/>
+        <mesh filename="package://ev3_manipulator/meshes/left_finger_inner_link_1.stl" scale="0.001 0.001 0.001"/>
       </geometry>
       <material name="silver"/>
@@ -202,5 +202,5 @@
       <origin xyz="0.04992 -0.305958 -0.147299" rpy="0 0 0"/>
       <geometry>
-        <mesh filename="file://$(find ev3_manipulator)/meshes/left_finger_inner_link_1.stl" scale="0.001 0.001 0.001"/>
+        <mesh filename="package://ev3_manipulator/meshes/left_finger_inner_link_1.stl" scale="0.001 0.001 0.001"/>
       </geometry>
     </collision>
@@ -216,5 +216,5 @@
       <origin xyz="-0.010062 -0.305958 -0.147299" rpy="0 0 0"/>
       <geometry>
-        <mesh filename="file://$(find ev3_manipulator)/meshes/left_finger_outer_link_1.stl" scale="0.001 0.001 0.001"/>
+        <mesh filename="package://ev3_manipulator/meshes/left_finger_outer_link_1.stl" scale="0.001 0.001 0.001"/>
       </geometry>
       <material name="silver"/>
@@ -223,5 +223,5 @@
       <origin xyz="-0.010062 -0.305958 -0.147299" rpy="0 0 0"/>
       <geometry>
-        <mesh filename="file://$(find ev3_manipulator)/meshes/left_finger_outer_link_1.stl" scale="0.001 0.001 0.001"/>
+        <mesh filename="package://ev3_manipulator/meshes/left_finger_outer_link_1.stl" scale="0.001 0.001 0.001"/>
       </geometry>
     </collision>
@@ -237,5 +237,5 @@
       <origin xyz="0.04992 -0.281275 -0.147299" rpy="0 0 0"/>
       <geometry>
-        <mesh filename="file://$(find ev3_manipulator)/meshes/right_finger_inner_link_1.stl" scale="0.001 0.001 0.001"/>
+        <mesh filename="package://ev3_manipulator/meshes/right_finger_inner_link_1.stl" scale="0.001 0.001 0.001"/>
       </geometry>
       <material name="silver"/>
@@ -244,5 +244,5 @@
       <origin xyz="0.04992 -0.281275 -0.147299" rpy="0 0 0"/>
       <geometry>
-        <mesh filename="file://$(find ev3_manipulator)/meshes/right_finger_inner_link_1.stl" scale="0.001 0.001 0.001"/>
+        <mesh filename="package://ev3_manipulator/meshes/right_finger_inner_link_1.stl" scale="0.001 0.001 0.001"/>
       </geometry>
     </collision>
@@ -258,5 +258,5 @@
       <origin xyz="-0.010062 -0.281275 -0.147299" rpy="0 0 0"/>
       <geometry>
-        <mesh filename="file://$(find ev3_manipulator)/meshes/right_finger_outer_link_1.stl" scale="0.001 0.001 0.001"/>
+        <mesh filename="package://ev3_manipulator/meshes/right_finger_outer_link_1.stl" scale="0.001 0.001 0.001"/>
       </geometry>
       <material name="silver"/>
@@ -265,5 +265,5 @@
       <origin xyz="-0.010062 -0.281275 -0.147299" rpy="0 0 0"/>
       <geometry>
-        <mesh filename="file://$(find ev3_manipulator)/meshes/right_finger_outer_link_1.stl" scale="0.001 0.001 0.001"/>
+        <mesh filename="package://ev3_manipulator/meshes/right_finger_outer_link_1.stl" scale="0.001 0.001 0.001"/>
       </geometry>
     </collision>
@@ -282,5 +282,5 @@
       <origin xyz="0.073638 -0.18132 -0.03" rpy="0 0 0"/>
       <geometry>
-        <mesh filename="file://$(find ev3_manipulator)/meshes/base_motor_housing_linkage_1.stl" scale="0.001 0.001 0.001"/>
+        <mesh filename="package://ev3_manipulator/meshes/base_motor_housing_linkage_1.stl" scale="0.001 0.001 0.001"/>
       </geometry>
       <material name="silver"/>
@@ -289,5 +289,5 @@
       <origin xyz="0.073638 -0.18132 -0.03" rpy="0 0 0"/>
       <geometry>
-        <mesh filename="file://$(find ev3_manipulator)/meshes/base_motor_housing_linkage_1.stl" scale="0.001 0.001 0.001"/>
+        <mesh filename="package://ev3_manipulator/meshes/base_motor_housing_linkage_1.stl" scale="0.001 0.001 0.001"/>
       </geometry>
     </collision>
@@ -303,5 +303,5 @@
       <origin xyz="0.05 -0.18875 -0.07" rpy="0 0 0"/>
       <geometry>
-        <mesh filename="file://$(find ev3_manipulator)/meshes/motor_housing_link_1.stl" scale="0.001 0.001 0.001"/>
+        <mesh filename="package://ev3_manipulator/meshes/motor_housing_link_1.stl" scale="0.001 0.001 0.001"/>
       </geometry>
       <material name="silver"/>
@@ -310,5 +310,5 @@
       <origin xyz="0.05 -0.18875 -0.07" rpy="0 0 0"/>
       <geometry>
-        <mesh filename="file://$(find ev3_manipulator)/meshes/motor_housing_link_1.stl" scale="0.001 0.001 0.001"/>
+        <mesh filename="package://ev3_manipulator/meshes/motor_housing_link_1.stl" scale="0.001 0.001 0.001"/>
       </geometry>
     </collision>
@@ -324,5 +324,5 @@
       <origin xyz="0.152651 -0.33625 -0.052373" rpy="0 0 0"/>
       <geometry>
-        <mesh filename="file://$(find ev3_manipulator)/meshes/bench_stand_link_1.stl" scale="0.001 0.001 0.001"/>
+        <mesh filename="package://ev3_manipulator/meshes/bench_stand_link_1.stl" scale="0.001 0.001 0.001"/>
       </geometry>
       <material name="silver"/>
@@ -331,5 +331,5 @@
       <origin xyz="0.152651 -0.33625 -0.052373" rpy="0 0 0"/>
       <geometry>
-        <mesh filename="file://$(find ev3_manipulator)/meshes/bench_stand_link_1.stl" scale="0.001 0.001 0.001"/>
+        <mesh filename="package://ev3_manipulator/meshes/bench_stand_link_1.stl" scale="0.001 0.001 0.001"/>
       </geometry>
     </collision>
@@ -345,5 +345,5 @@
       <origin xyz="0.152314 -0.341622 -0.064322" rpy="0 0 0"/>
       <geometry>
-        <mesh filename="file://$(find ev3_manipulator)/meshes/sensor_housing_link_1.stl" scale="0.001 0.001 0.001"/>
+        <mesh filename="package://ev3_manipulator/meshes/sensor_housing_link_1.stl" scale="0.001 0.001 0.001"/>
       </geometry>
       <material name="silver"/>
@@ -352,5 +352,5 @@
       <origin xyz="0.152314 -0.341622 -0.064322" rpy="0 0 0"/>
       <geometry>
-        <mesh filename="file://$(find ev3_manipulator)/meshes/sensor_housing_link_1.stl" scale="0.001 0.001 0.001"/>
+        <mesh filename="package://ev3_manipulator/meshes/sensor_housing_link_1.stl" scale="0.001 0.001 0.001"/>
       </geometry>
     </collision>
@@ -366,5 +366,5 @@
       <origin xyz="-0.12 -0.16875 -0.03" rpy="0 0 0"/>
       <geometry>
-        <mesh filename="file://$(find ev3_manipulator)/meshes/conveyor_base_linkage_1.stl" scale="0.001 0.001 0.001"/>
+        <mesh filename="package://ev3_manipulator/meshes/conveyor_base_linkage_1.stl" scale="0.001 0.001 0.001"/>
       </geometry>
       <material name="silver"/>
@@ -373,5 +373,5 @@
       <origin xyz="-0.12 -0.16875 -0.03" rpy="0 0 0"/>
       <geometry>
-        <mesh filename="file://$(find ev3_manipulator)/meshes/conveyor_base_linkage_1.stl" scale="0.001 0.001 0.001"/>
+        <mesh filename="package://ev3_manipulator/meshes/conveyor_base_linkage_1.stl" scale="0.001 0.001 0.001"/>
       </geometry>
     </collision>
@@ -387,5 +387,5 @@
       <origin xyz="0.1029 -0.24175 -0.0329" rpy="0 0 0"/>
       <geometry>
-        <mesh filename="file://$(find ev3_manipulator)/meshes/conveyor_linkage_link_1.stl" scale="0.001 0.001 0.001"/>
+        <mesh filename="package://ev3_manipulator/meshes/conveyor_linkage_link_1.stl" scale="0.001 0.001 0.001"/>
       </geometry>
       <material name="silver"/>
@@ -394,5 +394,5 @@
       <origin xyz="0.1029 -0.24175 -0.0329" rpy="0 0 0"/>
       <geometry>
-        <mesh filename="file://$(find ev3_manipulator)/meshes/conveyor_linkage_link_1.stl" scale="0.001 0.001 0.001"/>
+        <mesh filename="package://ev3_manipulator/meshes/conveyor_linkage_link_1.stl" scale="0.001 0.001 0.001"/>
       </geometry>
     </collision>
@@ -408,5 +408,5 @@
       <origin xyz="0.1029 -0.25575 -0.0329" rpy="0 0 0"/>
       <geometry>
-        <mesh filename="file://$(find ev3_manipulator)/meshes/conveyor_belt_link_1.stl" scale="0.001 0.001 0.001"/>
+        <mesh filename="package://ev3_manipulator/meshes/conveyor_belt_link_1.stl" scale="0.001 0.001 0.001"/>
       </geometry>
       <material name="silver"/>
@@ -415,5 +415,5 @@
       <origin xyz="0.1029 -0.25575 -0.0329" rpy="0 0 0"/>
       <geometry>
-        <mesh filename="file://$(find ev3_manipulator)/meshes/conveyor_belt_link_1.stl" scale="0.001 0.001 0.001"/>
+        <mesh filename="package://ev3_manipulator/meshes/conveyor_belt_link_1.stl" scale="0.001 0.001 0.001"/>
       </geometry>
     </collision>
@@ -429,5 +429,5 @@
       <origin xyz="0.173678 -0.24175 -0.052322" rpy="0 0 0"/>
       <geometry>
-        <mesh filename="file://$(find ev3_manipulator)/meshes/left_motor_shaft_link_1.stl" scale="0.001 0.001 0.001"/>
+        <mesh filename="package://ev3_manipulator/meshes/left_motor_shaft_link_1.stl" scale="0.001 0.001 0.001"/>
       </geometry>
       <material name="silver"/>
@@ -436,5 +436,5 @@
       <origin xyz="0.173678 -0.24175 -0.052322" rpy="0 0 0"/>
       <geometry>
-        <mesh filename="file://$(find ev3_manipulator)/meshes/left_motor_shaft_link_1.stl" scale="0.001 0.001 0.001"/>
+        <mesh filename="package://ev3_manipulator/meshes/left_motor_shaft_link_1.stl" scale="0.001 0.001 0.001"/>
       </geometry>
     </collision>
@@ -450,5 +450,5 @@
       <origin xyz="0.173678 -0.27575 -0.052322" rpy="0 0 0"/>
       <geometry>
-        <mesh filename="file://$(find ev3_manipulator)/meshes/right_pulley_link_1.stl" scale="0.001 0.001 0.001"/>
+        <mesh filename="package://ev3_manipulator/meshes/right_pulley_link_1.stl" scale="0.001 0.001 0.001"/>
       </geometry>
       <material name="silver"/>
@@ -457,5 +457,5 @@
       <origin xyz="0.173678 -0.27575 -0.052322" rpy="0 0 0"/>
       <geometry>
-        <mesh filename="file://$(find ev3_manipulator)/meshes/right_pulley_link_1.stl" scale="0.001 0.001 0.001"/>
+        <mesh filename="package://ev3_manipulator/meshes/right_pulley_link_1.stl" scale="0.001 0.001 0.001"/>
       </geometry>
     </collision>
@@ -471,5 +471,5 @@
       <origin xyz="-0.166124 -0.26175 -0.052322" rpy="0 0 0"/>
       <geometry>
-        <mesh filename="file://$(find ev3_manipulator)/meshes/right_pulley_shaft_link_1.stl" scale="0.001 0.001 0.001"/>
+        <mesh filename="package://ev3_manipulator/meshes/right_pulley_shaft_link_1.stl" scale="0.001 0.001 0.001"/>
       </geometry>
       <material name="silver"/>
@@ -478,5 +478,5 @@
       <origin xyz="-0.166124 -0.26175 -0.052322" rpy="0 0 0"/>
       <geometry>
-        <mesh filename="file://$(find ev3_manipulator)/meshes/right_pulley_shaft_link_1.stl" scale="0.001 0.001 0.001"/>
+        <mesh filename="package://ev3_manipulator/meshes/right_pulley_shaft_link_1.stl" scale="0.001 0.001 0.001"/>
       </geometry>
     </collision>
@@ -492,5 +492,5 @@
       <origin xyz="-0.166124 -0.27575 -0.052322" rpy="0 0 0"/>
       <geometry>
-        <mesh filename="file://$(find ev3_manipulator)/meshes/right_pulley_link1_1.stl" scale="0.001 0.001 0.001"/>
+        <mesh filename="package://ev3_manipulator/meshes/right_pulley_link1_1.stl" scale="0.001 0.001 0.001"/>
       </geometry>
       <material name="silver"/>
@@ -499,5 +499,5 @@
       <origin xyz="-0.166124 -0.27575 -0.052322" rpy="0 0 0"/>
       <geometry>
-        <mesh filename="file://$(find ev3_manipulator)/meshes/right_pulley_link1_1.stl" scale="0.001 0.001 0.001"/>
+        <mesh filename="package://ev3_manipulator/meshes/right_pulley_link1_1.stl" scale="0.001 0.001 0.001"/>
       </geometry>
     </collision>
