Commit message: update digital-twin launch, urdf, and controller config for conveyor plugin

File: mani_digital_ev3/urdf/manipulator_gazebo.xacro (robot description, xacro)
@@ -50,7 +50,5 @@
   <!-- ══════════════════════════════════════════════════════════════
        GRIPPER — gears + fingers
-       Finger contact links carry a low-slip friction surface.
-       self_collide=false on moving gripper links to avoid the fingers
-       fighting each other in contact (a common Gazebo gripper jam).
+       Friction coefficients elevated to keep ball locked in grasp
   ══════════════════════════════════════════════════════════════ -->
   <gazebo reference="left_gear_1">
@@ -68,65 +66,25 @@
   <gazebo reference="left_inner_finger_1">
     <material>${body_color}</material>
-    <self_collide>false</self_collide>
-    <collision name="left_inner_finger_1_collision">
-      <surface>
-        <friction>
-          <ode>
-            <mu>0.1</mu>
-            <mu2>0.1</mu2>
-            <slip1>0.05</slip1>
-            <slip2>0.05</slip2>
-          </ode>
-        </friction>
-      </surface>
-    </collision>
+    <mu1>1.5</mu1>
+    <mu2>1.5</mu2>
+    <self_collide>false</self_collide>
   </gazebo>
   <gazebo reference="left_outer_finger_1">
     <material>${body_color}</material>
-    <self_collide>false</self_collide>
-    <collision name="left_outer_finger_1_collision">
-      <surface>
-        <friction>
-          <ode>
-            <mu>0.1</mu>
-            <mu2>0.1</mu2>
-            <slip1>0.05</slip1>
-            <slip2>0.05</slip2>
-          </ode>
-        </friction>
-      </surface>
-    </collision>
+    <mu1>1.5</mu1>
+    <mu2>1.5</mu2>
+    <self_collide>false</self_collide>
   </gazebo>
   <gazebo reference="right_inner_finger_1">
     <material>${body_color}</material>
-    <self_collide>false</self_collide>
-    <collision name="right_inner_finger_1_collision">
-      <surface>
-        <friction>
-          <ode>
-            <mu>0.1</mu>
-            <mu2>0.1</mu2>
-            <slip1>0.05</slip1>
-            <slip2>0.05</slip2>
-          </ode>
-        </friction>
-      </surface>
-    </collision>
+    <mu1>1.5</mu1>
+    <mu2>1.5</mu2>
+    <self_collide>false</self_collide>
   </gazebo>
   <gazebo reference="right_outer_finger_1">
     <material>${body_color}</material>
-    <self_collide>false</self_collide>
-    <collision name="right_outer_finger_1_collision">
-      <surface>
-        <friction>
-          <ode>
-            <mu>0.1</mu>
-            <mu2>0.1</mu2>
-            <slip1>0.05</slip1>
-            <slip2>0.05</slip2>
-          </ode>
-        </friction>
-      </surface>
-    </collision>
+    <mu1>1.5</mu1>
+    <mu2>1.5</mu2>
+    <self_collide>false</self_collide>
   </gazebo>
   <gazebo reference="motor_shaft_arm_4_outer_gripper_1">
@@ -147,6 +105,6 @@
   <gazebo reference="conveyor_belt_link_1">
     <material>${body_color}</material>
-    <mu1>0.8</mu1>
-    <mu2>0.8</mu2>
+    <mu1>1.0</mu1>
+    <mu2>1.0</mu2>
     <self_collide>false</self_collide>
   </gazebo>
@@ -205,9 +163,41 @@
     <self_collide>false</self_collide>
   </gazebo>
-  <!-- ══════════════════════════════════════════════════════════════
-       gz_ros2_control plugin — kept exactly as the working setup
-       (Humble + Ignition Fortress). Only the controller.yaml path and
-       the global fallback gain live here.
-  ══════════════════════════════════════════════════════════════ -->
+  <gazebo reference="belt_moving">
+    <!-- Friction between the belt surface and ball -->
+    <mu1>1.5</mu1>
+    <mu2>1.5</mu2>
+    <!-- Contact stability -->
+    <kp>1000000.0</kp>
+    <kd>10.0</kd>
+    <minDepth>0.0001</minDepth>
+    <maxVel>0.1</maxVel>
+    <!-- Debug colour -->
+    <material>Gazebo/Red</material>
+  </gazebo>
+  <!-- ══════════════════════════════════════════════════════════════
+       PLUGINS (IGNITION GAZEBO FORTRESS)
+  ══════════════════════════════════════════════════════════════ -->
+  <!-- IFRA Conveyor Belt Plugin for Ignition Gazebo Fortress -->
+  <!-- <gazebo>
+    <plugin
+      filename="libconveyorbelt_gazebo.so"
+      name="conveyorbelt_gazebo::ConveyorBeltPlugin">
+      <max_velocity>1.0</max_velocity>
+      <belt_link>conveyor_belt_link_1</belt_link>
+    </plugin>
+  </gazebo> -->
+  <gazebo>
+    <plugin
+      name="ros2_conveyorbelt_system"
+      filename="libros2gz_conveyorbelt_system.so">
+      <max_velocity>1.0</max_velocity>
+      <publish_rate>1000</publish_rate>
+      <!-- This refers to the separately declared prismatic joint. -->
+      <joint_name>belt_joint</joint_name>
+      <lower_limit>0.0</lower_limit>
+      <upper_limit>0.01</upper_limit>
+    </plugin>
+  </gazebo>
+  <!-- gz_ros2_control plugin -->
   <gazebo>
     <plugin filename="gz_ros2_control-system"

File: mani_digital_ev3/urdf/manipulator_urdf.xacro (robot description, xacro)
@@ -1,4 +1,10 @@
 <?xml version='1.0' encoding='UTF-8'?>
 <robot xmlns:xacro="http://www.ros.org/wiki/xacro" name="mani_digital_ev3">
+    <xacro:property name="belt_surface_length" value="0.34"/>
+    <xacro:property name="belt_surface_width" value="0.05"/>
+    <xacro:property name="belt_surface_thickness" value="0.001"/>
+    <xacro:property name="belt_surface_x" value="0.102917"/>
+    <xacro:property name="belt_surface_y" value="0.083295"/>
+    <xacro:property name="belt_surface_z" value="0.033500"/>
     <!-- ══════════════════════════════════════════════════════════════════════
         WORLD ANCHOR — fixes base_link so the arm does not drift/fall.
@@ -513,4 +519,51 @@
       </collision>
     </link>
+    <!-- ================================================================
+     THIN MOVING CONTACT SURFACE
+================================================================ -->
+<link name="belt_moving">
+  <inertial>
+    <origin xyz="0 0 0" rpy="0 0 0"/>
+    <mass value="0.1"/>
+    <!--
+      Approximate box inertia for:
+          mass = 0.1 kg
+          size = 0.34 x 0.05 x 0.001 m
+    -->
+    <inertia
+      ixx="0.00002084"
+      iyy="0.00096334"
+      izz="0.00098417"
+      ixy="0"
+      ixz="0"
+      iyz="0"/>
+  </inertial>
+  <collision>
+    <origin xyz="0 0 0" rpy="0 0 0"/>
+    <geometry>
+      <box
+        size="${belt_surface_length}
+              ${belt_surface_width}
+              ${belt_surface_thickness}"/>
+    </geometry>
+  </collision>
+  <!--
+    Temporary debug visual.
+    It should appear as a thin red transparent plate over the conveyor.
+    Remove this visual after confirming the alignment.
+  -->
+  <visual>
+    <origin xyz="0 0 0" rpy="0 0 0"/>
+    <geometry>
+      <box
+        size="${belt_surface_length}
+              ${belt_surface_width}
+              ${belt_surface_thickness}"/>
+    </geometry>
+    <material name="belt_moving_debug_material">
+      <color rgba="1.0 0.0 0.0 0.45"/>
+    </material>
+  </visual>
+</link>
     <!-- ══════════════════════════════════════════════════════════════════════
         ARM JOINTS (driven + parallelogram mimic)
@@ -698,3 +751,29 @@
       <child link="conveyor_belt_link_1"/>
     </joint>
+<!-- ================================================================
+     MOVING CONVEYOR SURFACE JOINT
+================================================================ -->
+    <joint name="belt_joint" type="prismatic">
+      <parent link="conveyor_belt_link_1"/>
+      <child link="belt_moving"/>
+      <!--
+        Approximate world position of the moving surface centre:
+          X = -0.102917 + 0.102917 = 0.0
+          Y =  0.149705 + 0.083295 = 0.233
+          Z =  0.010000 + 0.033500 = 0.0435
+      -->
+      <origin
+        xyz="${belt_surface_x} ${belt_surface_y} ${belt_surface_z}"
+        rpy="0 0 0"/>
+      <!-- Belt transport direction -->
+      <axis xyz="1 0 0"/>
+      <limit
+        lower="0.0"
+        upper="0.01"
+        effort="100000000.0"
+        velocity="10.0"/>
+      <dynamics
+        damping="1.0"
+        friction="0.0"/>
+    </joint>
 </robot>
